File: pcb_manu.kicad_sch (KiCad schematic)
At the start: 4 parts, among them J1 BATTERY, J2 SENSOR, U1 HT7333-A, U2 ESP32-WROOM-32

Commit message: feat: pcb v1
Parts:
- removed J1: BATTERY, symbol Conn_01x02
- removed J2: SENSOR, symbol Conn_01x03
- removed U1: HT7333-A, symbol HT7333-A
- removed U2: ESP32-WROOM-32, symbol ESP32-WROOM-32
- added C_Filtro1, C_Filtro2: 10uF, Capacitor_THT:C_Disc_D5.0mm_W2.5mm_P5.00mm, symbol Device:C
- added ESP32_C3: Conn_02x15_Counter_Clockwise, RF_Module:ESP32-C3-DevKitM-1, symbol Connector_Generic:Conn_02x15_Counter_Clockwise
- added J1: Conn_01x03_Pin, Connector_JST:JST_XH_B3B-XH-AM_1x03_P2.50mm_Vertical, symbol Connector:Conn_01x03_Pin
- added Regulador1: MCP1700x-330xxMB, Package_TO_SOT_THT:TO-92S, symbol Regulator_Linear:MCP1700x-330xxMB
- added TP1, TP2: TestPoint, TestPoint:TestPoint_Bridge_Pitch2.54mm_Drill0.7mm, symbol Connector:TestPoint
Connections:
- net 3V3: now also C_Filtro1.1, ESP32_C3.1 (Pin_1), J1.3 (Pin_3), Regulador1.3 (VO)
- net GND: now also C_Filtro1.2, C_Filtro2.2, ESP32_C3.29 (Pin_29), J1.2 (Pin_2), Regulador1.1 (GND), TP1.1
- net Vin: now also C_Filtro2.1, Regulador1.2 (VI), TP2.1
- new net D34: ESP32_C3.19 (Pin_19), J1.1 (Pin_1)
Other:
- company: Antigravity Design -> Fernando Román
- title: PCB Manu - ESP32 Soil Sensor -> ESP32 Soil Sensor
